Commit message: used dwa_local_planner

File: src/mecanum_sim/urdf/mecanum.xacro (robot description, xacro)
@@ -12,5 +12,5 @@
   <xacro:property name="lidar_width" value="0.0508" />    <!-- 2.0 in  -->
   <xacro:property name="lidar_length" value="0.0508" />    <!-- 2.0 in  -->
-  <xacro:property name="lidar_height" value="0.0762" />    <!-- 3.0 in  -->
+  <xacro:property name="lidar_height" value="0.1400" />    <!-- 3.0 in  -->
   <xacro:property name="lidar_setback" value="0.0127" />    <!-- 0.5 in  -->
   <!--~~~~~~~~~~~~~~~~~~~~~~~~ ~ ROBOT BASE ~ ~~~~~~~~~~~~~~~~~~~~~~~~~~~~~~-->
